Commit message: first commit

File: mars_ws/src/mars_lite_description/urdf/mars_lite_with_gripper.urdf.xacro (robot description, xacro)
@@ -102,35 +102,4 @@
   <xacro:caster_support prefix="back_left" reflect_fr="-1" reflect_lr="1"/>
   <xacro:caster_support prefix="back_right" reflect_fr="-1" reflect_lr="-1"/>
-  <!-- <xacro:macro name="caster_support" params="prefix reflect_fr reflect_lr">
-    <link name="${prefix}_caster_support">
-      <collision>
-          <origin xyz="0 0 ${-wheel_radius * 1.95}" rpy="0 0 0" />
-          <geometry>
-            <cylinder radius="0.025" length="${wheel_radius * 2}"/>
-          </geometry>
-        </collision>
-      <inertial>
-        <origin xyz="0 0 ${-wheel_radius * 2}" rpy="0 0 0" />
-        <mass value="1.0" />
-        <xacro:cylinder_inertia m="1.0" r="0.025" h="${wheel_radius * 2}" />
-      </inertial>
-    </link>
-    <joint name="${prefix}_caster_support_joint" type="fixed">
-      <origin xyz="${0.225 * reflect_fr} ${0.17 * reflect_lr} ${wheel_radius * 2}" rpy="0 0 0" />
-      <parent link="base_link"/>
-      <child link="${prefix}_caster_support"/>
-    </joint>
-    <gazebo reference="${prefix}_caster_support">
-        <mu1 value="0.01"/>
-        <mu2 value="0.01"/>
-        <kp  value="1000000.0" />
-        <kd  value="10000.0" />
-        <fdir1 value="1 0 0" />
-    </gazebo>
-  </xacro:macro>
-  <xacro:caster_support prefix="front_left" reflect_fr="1" reflect_lr="1"/>
-  <xacro:caster_support prefix="front_right" reflect_fr="1" reflect_lr="-1"/>
-  <xacro:caster_support prefix="back_left" reflect_fr="-1" reflect_lr="1"/>
-  <xacro:caster_support prefix="back_right" reflect_fr="-1" reflect_lr="-1"/> -->
   <!-- Driving wheels -->
   <xacro:macro name="wheel" params="prefix reflect">

File: mars_ws/src/tmr_ros1_simplified_edition/tm5_description/urdf/tm5_700.urdf.xacro (robot description, xacro)
@@ -33,10 +33,10 @@
     <!-- Inertia parameters -->
     <xacro:property name="base_mass" value="1.0" />
-    <xacro:property name="shoulder_mass" value="4.5" />
-    <xacro:property name="arm_1_mass" value="11.0" />
-    <xacro:property name="arm_2_mass" value="2.5" />
-    <xacro:property name="wrist_1_mass" value="1.45" />
-    <xacro:property name="wrist_2_mass" value="1.45" />
-    <xacro:property name="wrist_3_mass" value="0.4" />
+    <xacro:property name="shoulder_mass" value="4.032" />
+    <xacro:property name="arm_1_mass" value="8.567" />
+    <xacro:property name="arm_2_mass" value="2.273" />
+    <xacro:property name="wrist_1_mass" value="1.576" />
+    <xacro:property name="wrist_2_mass" value="1.576" />
+    <xacro:property name="wrist_3_mass" value="0.31" />
     <!-- Kinematic model -->
     <!-- Properties from tmcontrol.conf -->

Commit message: add shoppingmall world and scene map builder

File: mars_ws/src/mars_lite_description/urdf/mars_lite_with_gripper.urdf.xacro (robot description, xacro)
@@ -4,4 +4,5 @@
   <xacro:arg name="laser_enabled" default="1" />
   <xacro:arg name="realsense_enabled" default="0" />
+  <xacro:arg name="imu_enabled" default="0" />
   <!-- Gazebo plugin -->
   <xacro:include filename="$(find mars_lite_description)/urdf/mars_lite.gazebo" />
@@ -220,3 +221,119 @@
     <origin xyz="0 0 0" rpy="${-pi / 2} ${-pi / 2} 0"/>
   </xacro:robotiq_85_gripper>
+  <!-- IMU -->
+  <!-- <xacro:if value="$(arg imu_enabled)">
+  <xacro:include filename="$(find mars_lite_description)/urdf/accessories/intel_realsense.urdf.xacro"/>
+    <xacro:intel_realsense_mount prefix="camera1" topic="camera1" parent_link="realsense_mount"/>
+    <link name="realsense_mount"/>
+    <joint name="realsense_mount_joint" type="fixed">
+      <origin xyz="0 0.05 0.062" rpy="0 ${-pi / 2} ${-pi / 2}" />
+      <parent link="tm_wrist_3_link"/>
+      <child link="realsense_mount" />
+    </joint>
+  </xacro:if>
+  <sensor name="imu_sensor" type="imu">
+      <always_on>true</always_on>
+      <update_rate>100</update_rate>
+      <visualize>true</visualize>
+      <topic>imu</topic>
+      <plugin filename="libgazebo_ros_imu_sensor.so" name="imu_plugin">
+        <topicName>imu</topicName>
+        <bodyName>base_link</bodyName>
+        <updateRateHZ>100.0</updateRateHZ>
+        <gaussianNoise>0.0</gaussianNoise>
+        <xyzOffset>0 0 0</xyzOffset>
+        <rpyOffset>0 0 0</rpyOffset>
+        <frameName>imu_link</frameName>
+      </plugin>
+      <pose>0 0 0 0 0 0</pose>
+    </sensor> -->
+  <!-- <xacro:macro name="imu" params="imu">
+    <joint name="imu_joint" type="fixed">
+      <axis xyz="1 0 0"/>
+      <origin xyz="0 0 0.19"/>
+      <parent link="base_link"/>
+      <child link="imu_link"/>
+    </joint>
+    <link name="imu_link">
+      <inertial>
+        <mass value="0.001"/>
+        <origin rpy="0 0 0" xyz="0 0 0"/>
+        <inertia ixx="0.0001" ixy="0" ixz="0" iyy="0.000001" iyz="0" izz="0.0001"/>
+      </inertial>
+      <visual>
+        <origin rpy="0 0 0" xyz="0 0 0"/>
+        <geometry>
+          <box size="0.001 0.001 0.001"/>
+        </geometry>
+      </visual>
+      <collision>
+        <origin rpy="0 0 0" xyz="0 0 0"/>
+        <geometry>
+          <box size=".001 .001 .001"/>
+        </geometry>
+      </collision>
+    </link>
+    <gazebo>
+    <plugin name="imu_plugin" filename="libgazebo_ros_imu.so">
+      <alwaysOn>true</alwaysOn>
+      <bodyName>imu_link</bodyName>
+      <topicName>imu</topicName>
+      <serviceName>imu_service</serviceName>
+      <gaussianNoise>0.0</gaussianNoise>
+      <updateRate>0</updateRate>
+      <imu>
+        <noise>
+          <type>gaussian</type>
+          <rate>
+            <mean>0.0</mean>
+            <stddev>2e-4</stddev>
+            <bias_mean>0.0000075</bias_mean>
+            <bias_stddev>0.0000008</bias_stddev>
+          </rate>
+          <accel>
+            <mean>0.0</mean>
+            <stddev>1.7e-2</stddev>
+            <bias_mean>0.1</bias_mean>
+            <bias_stddev>0.001</bias_stddev>
+          </accel>
+        </noise>
+      </imu>
+    </plugin>
+  </gazebo>
+  </xacro:macro> -->
+  <!-- <gazebo reference="imu_link">
+    <sensor type="imu" name="imu">
+      <always_on>true</always_on>
+      <visualize>$(arg imu_visual)</visualize>
+    </sensor>
+    <material>Gazebo/Grey</material>
+  </gazebo> -->
+  <gazebo>
+    <plugin name="imu_plugin" filename="libgazebo_ros_imu.so">
+      <alwaysOn>true</alwaysOn>
+      <bodyName>base_link</bodyName>
+      <frameName>base_link</frameName>
+      <topicName>imu</topicName>
+      <serviceName>imu_service</serviceName>
+      <gaussianNoise>0.0</gaussianNoise>
+      <updateRate>0</updateRate>
+      <imu>
+        <noise>
+          <type>gaussian</type>
+          <rate>
+            <mean>0.0</mean>
+            <stddev>2e-4</stddev>
+            <bias_mean>0.0000075</bias_mean>
+            <bias_stddev>0.0000008</bias_stddev>
+          </rate>
+          <accel>
+            <mean>0.0</mean>
+            <stddev>1.7e-2</stddev>
+            <bias_mean>0.1</bias_mean>
+            <bias_stddev>0.001</bias_stddev>
+          </accel>
+        </noise>
+      </imu>
+    </plugin>
+  </gazebo>
 </robot>

Commit message: code clean up

File: mars_ws/src/mars_lite_description/urdf/mars_lite_with_gripper.urdf.xacro (robot description, xacro)
@@ -309,5 +309,38 @@
     <material>Gazebo/Grey</material>
   </gazebo> -->
+  <joint name="imu_joint" type="fixed">
+    <parent link="base_link"/>
+    <child link="imu_link"/>
+    <origin xyz="-0.032 0 0.068" rpy="0 0 0"/>
+  </joint>
+  <link name="imu_link"/>
   <gazebo>
+    <plugin name="imu_plugin" filename="libgazebo_ros_imu.so">
+      <alwaysOn>true</alwaysOn>
+      <bodyName>imu_link</bodyName>
+      <topicName>imu</topicName>
+      <serviceName>imu_service</serviceName>
+      <gaussianNoise>0.0</gaussianNoise>
+      <updateRate>0</updateRate>
+      <imu>
+        <noise>
+          <type>gaussian</type>
+          <rate>
+            <mean>0.0</mean>
+            <stddev>2e-4</stddev>
+            <bias_mean>0.0000075</bias_mean>
+            <bias_stddev>0.0000008</bias_stddev>
+          </rate>
+          <accel>
+            <mean>0.0</mean>
+            <stddev>1.7e-2</stddev>
+            <bias_mean>0.1</bias_mean>
+            <bias_stddev>0.001</bias_stddev>
+          </accel>
+        </noise>
+      </imu>
+    </plugin>
+  </gazebo>
+  <!-- <gazebo>
     <plugin name="imu_plugin" filename="libgazebo_ros_imu.so">
       <alwaysOn>true</alwaysOn>
@@ -336,4 +369,4 @@
       </imu>
     </plugin>
-  </gazebo>
+  </gazebo> -->
 </robot>
